Commit message: Lab 2 end

File: dh2urdf/urdf/dynamic.urdf (robot description, URDF)
Before this commit: robot manipulator, 4 links, 3 joints
Links:
- added link join2; visual sphere radius=0.2
- added link join3; visual sphere radius=0.2
- added link left_gripper; visual mesh filename=package://dh2urdf/meshes/l_finger.dae
- added link left_tip; visual mesh filename=package://dh2urdf/meshes/l_finger_tip.dae
- added link right_gripper; visual mesh filename=package://dh2urdf/meshes/l_finger.dae
- added link right_tip; visual mesh filename=package://dh2urdf/meshes/l_finger_tip.dae
- link base_link: geometry visual cylinder length=0.04 radius=0.15
- link link_1: geometry visual cylinder length=${props['i1']['l_len']} radius=0.05
- link link_2: geometry visual cylinder length=${props['i2']['l_len']} radius=0.05
- link link_3: geometry visual cylinder length=${props['i3']['l_len']} radius=0.05
Joints:
- removed joint link1_to_link2
- removed joint link2_to_link3
- added joint join2_to_link2: type continuous, parent join2, child link_2, origin xyz=0 0 0 rpy=0 0 0, axis 0 0 1
- added joint join3_to_link3: type fixed, parent join3, child link_3, origin xyz=${props['i3']['j_xyz']} rpy=${props['i3']['j_rpy']}, axis 0 0 1
- added joint left_gripper_joint: type fixed, parent link_3, child left_gripper, origin xyz=0 0.01 0 rpy=0 0 0
- added joint left_tip_joint: type fixed, parent left_gripper, child left_tip
- added joint link1_to_join2: type fixed, parent link_1, child join2, origin xyz=${props['i1']['j_xyz']} rpy=${props['i1']['j_rpy']}, axis 0 0 1
- added joint link2_to_join3: type continuous, parent link_2, child join3, origin xyz=${props['i2']['j_xyz']} rpy=${props['i2']['j_rpy']}, axis 0 0 1
- added joint right_gripper_joint: type fixed, parent link_3, child right_gripper, origin xyz=0 -0.01 0 rpy=0 0 0
- added joint right_tip_joint: type fixed, parent right_gripper, child right_tip
- joint base_to_link1: limit lower=-1.57075 upper=1.57075 effort=1000.0 velocity=0.5 -> lower=-${props['i1']['l_len']} upper=0 effort=1000.0 velocity=0.5; origin xyz=${props['i1']['j_xyz']} rpy=${props['i1']['j_rpy']} -> xyz=0 0 0 rpy=0 0 0; type revolute -> prismatic

File: dh2urdf/urdf/static.urdf (robot description, URDF)
Before this commit: robot manipulator, 4 links, 3 joints
Links:
- added link join2; visual sphere radius=0.2
- added link join3; visual sphere radius=0.2
- added link left_gripper; visual mesh filename=package://dh2urdf/meshes/l_finger.dae
- added link left_tip; visual mesh filename=package://dh2urdf/meshes/l_finger_tip.dae
- added link right_gripper; visual mesh filename=package://dh2urdf/meshes/l_finger.dae
- added link right_tip; visual mesh filename=package://dh2urdf/meshes/l_finger_tip.dae
- link base_link: geometry visual cylinder length=0.04 radius=0.15
- link link_1: geometry visual cylinder length=${props['i1']['l_len']} radius=0.05
- link link_2: geometry visual cylinder length=${props['i2']['l_len']} radius=0.05
- link link_3: geometry visual cylinder length=${props['i3']['l_len']} radius=0.05
Joints:
- removed joint link1_to_link2
- removed joint link2_to_link3
- added joint join2_to_link2: type fixed, parent join2, child link_2, origin xyz=0 0 0 rpy=0 0 0, axis 0 0 1
- added joint join3_to_link3: type fixed, parent join3, child link_3, origin xyz=${props['i3']['j_xyz']} rpy=${props['i3']['j_rpy']}, axis 0 0 1
- added joint left_gripper_joint: type fixed, parent link_3, child left_gripper, origin xyz=0 0.01 0 rpy=0 0 0
- added joint left_tip_joint: type fixed, parent left_gripper, child left_tip
- added joint link1_to_join2: type fixed, parent link_1, child join2, origin xyz=${props['i1']['j_xyz']} rpy=${props['i1']['j_rpy']}, axis 0 0 1
- added joint link2_to_join3: type fixed, parent link_2, child join3, origin xyz=${props['i2']['j_xyz']} rpy=${props['i2']['j_rpy']}, axis 0 0 1
- added joint right_gripper_joint: type fixed, parent link_3, child right_gripper, origin xyz=0 -0.01 0 rpy=0 0 0
- added joint right_tip_joint: type fixed, parent right_gripper, child right_tip
- joint base_to_link1: origin xyz=${props['i1']['j_xyz']} rpy=${props['i1']['j_rpy']} -> xyz=0 0 0 rpy=0 0 0
